File: PMSM Board v1.7/Power Stage/PowerStage.sch (EAGLE design)
At the start: 16 parts, among them U1 TPS73733-Q1_DRB_8, U2 TPS54240_DRC_10, U3 LP38692_NGG_6

Commit message: More switcher work.
Parts:
- added C6: 47uF\, SwitcherPowerStage:CAP
- added C7, C8, C9: 1uF, SwitcherPowerStage:CAP0805
- C3: value (none) -> .1uF
- C4, C5: device SwitcherPowerStage:CAP1210 -> SwitcherPowerStage:CAP0805
- R5: value 7.68k -> 59k
- R6: value 7.68k -> 10k
Connections:
- removed net N$8: R5.2, U$1.2
- new net N$9: R5.1, R6.2, U2.VSENSE
- new net VCC3V3: C9.1, U1.OUT
- new net VCC5V0: U1.EN, U1.IN, U3.SNS, U3.VOUT
- new net VCC5V5: C6.1, R5.2, U$1.2, U3.VEN, U3.VIN, U3.VIN_2
- net GND: now also C6.2, C7.2, C8.2, C9.2, R6.1, U1.EPAD, U1.GND, U3.GND
Other:
- moved on the sheet: C4, C5, D1, R4, U1, U2, U3

Commit message: rerouting PMSM Board
Connections:
- net GND: now also U3.7
- net VCC5V0: now also C8.1
- net VCC5V5: now also C7.1
Changed lines of the file:
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@@
 <label x="12.7" y="116.84" size="1.778" layer="95"/>
+</segment>
+<segment>
+<pinref part="U3" gate="A" pin="7"/>
+<wire x1="83.82" y1="86.36" x2="91.44" y2="86.36" width="0.1524" layer="91"/>
+<label x="86.36" y="86.36" size="1.778" layer="95"/>
 </segment>
 </net>
@@
 <segment>
 <pinref part="U3" gate="A" pin="VIN_2"/>
-<wire x1="25.4" y1="93.98" x2="48.26" y2="93.98" width="0.1524" layer="91"/>
+<wire x1="25.4" y1="93.98" x2="33.02" y2="93.98" width="0.1524" layer="91"/>
 <label x="22.86" y="93.98" size="1.778" layer="95"/>
+<pinref part="C7" gate="G$1" pin="1"/>
+<junction x="33.02" y="93.98"/>
+<wire x1="33.02" y1="93.98" x2="48.26" y2="93.98" width="0.1524" layer="91"/>
 </segment>
 <segment>
@@
 <label x="111.76" y="93.98" size="1.778" layer="95"/>
 <pinref part="U3" gate="A" pin="SNS"/>
-<wire x1="88.9" y1="93.98" x2="111.76" y2="93.98" width="0.1524" layer="91"/>
+<wire x1="88.9" y1="93.98" x2="99.06" y2="93.98" width="0.1524" layer="91"/>
+<wire x1="99.06" y1="93.98" x2="111.76" y2="93.98" width="0.1524" layer="91"/>
 <wire x1="83.82" y1="91.44" x2="88.9" y2="91.44" width="0.1524" layer="91"/>
 <wire x1="88.9" y1="91.44" x2="88.9" y2="93.98" width="0.1524" layer="91"/>
 <junction x="88.9" y="93.98"/>
+<pinref part="C8" gate="G$1" pin="1"/>
+<junction x="99.06" y="93.98"/>
 </segment>
 <segment>
@@
 <wire x1="15.24" y1="134.62" x2="15.24" y2="132.08" width="0.1524" layer="91"/>
 <pinref part="C9" gate="G$1" pin="1"/>
+<junction x="15.24" y="132.08"/>
 </segment>
 </net>
