File: PMSM Board v1.7/CANTensegrityBoard.sch (EAGLE design)
At the start: 74 parts, among them IC1 DRV8303, U10 H1206T500R-10, U2 SN65HVD232_D_8, U3 SN65LVDT348_PW_1, U9 H1206T500R-10

Commit message: rerouting PMSM Board
Parts:
- added C14: 5600pF, SwitcherPowerStage:CAP0805
- added C15: 270pF, SwitcherPowerStage:CAP0805
- added C29: 47uF\, SwitcherPowerStage:CAP
- added C30, C31, C32: 1uF, SwitcherPowerStage:CAP0805
- added C5: 4.7uF, SwitcherPowerStage:CAP1210
- added C6: .01uF, SwitcherPowerStage:CAP0805
- added C8: .1uF, SwitcherPowerStage:CAP0805
- added D1: DIODE-SCHOTTKY240A, SwitcherPowerStage:DIODE-SCHOTTKY240A
- added R10: 59k, SwitcherPowerStage:RESISTOR0805-RES
- added R11: 10k, SwitcherPowerStage:RESISTOR0805-RES
- added R2: 348k, SwitcherPowerStage:RESISTOR0805-RES
- added R3: 88.7k, SwitcherPowerStage:RESISTOR0805-RES
- added R8: 237k, SwitcherPowerStage:RESISTOR0805-RES
- added R9: 7.68k, SwitcherPowerStage:RESISTOR0805-RES
- added U$13: SLF12555T, SwitcherPowerStage:SLF12555T
- added U1: TPS73733-Q1_DRB_8, SwitcherPowerStage:TPS73733-Q1_DRB_8
- added U4: TPS54240_DRC_10, SwitcherPowerStage:TPS54240_DRC_10
- added U5: LP38692_NGG_6, SwitcherPowerStage:LP38692_NGG_6
- C2, C4: device ASL:CAP1206 -> ASL:CAP0805
Connections:
- new net N$10: C8.1, U4.BOOT
- new net N$13: C8.2, D1.C, U$13.1, U4.PH
- new net N$14: C15.1, R9.2, U4.COMP
- new net N$15: C14.1, R9.1
- new net N$16: R10.1, R11.2, U4.VSENSE
- new net N$7: R2.1, R3.2, U4.EN
- new net N$8: C6.1, U4.SS/TR
- new net N$9: R8.2, U4.RT/CLK
- new net VCC5V0: C31.1, U1.EN, U1.IN, U5.SNS, U5.VOUT
- new net VCC5V5: C29.1, C30.1, R10.2, U$13.2, U5.VEN, U5.VIN, U5.VIN_2
- net GND: now also C14.2, C15.2, C29.2, C30.2, C31.2, C32.2, C5.2, C6.2, D1.A, R11.1, R3.1, R8.1, U1.EPAD, U1.GND, U4.GND, U5.7, U5.GND
- net PVDD: now also C5.1, R2.2, U4.VIN
- net VCC3V3: now also C32.1, U1.OUT

Commit message: Started making room for connectors
Parts:
- removed C1: .1 uF 100V, ASL:CAP0805
- removed C2: 2.2uF 100V, ASL:CAP0805
Connections:
- removed net N$11: C9.2, IC1.SH_A
- removed net VCC5V: JP5.6
- net DRV_GND: no longer C1.2, C2.2
- net GND: no longer C14.2, C15.2, C29.2, C30.2, C31.2, C32.2, C5.2, C6.2, D1.A, R11.1, R3.1, R8.1, U1.EPAD, U1.GND, U4.GND, U5.7, U5.GND
- net PGND: now also C14.2, C15.2, C29.2, C30.2, C31.2, C32.2, C5.2, C6.2, D1.A, R11.1, R3.1, R8.1, U1.EPAD, U1.GND, U4.GND, U5.7, U5.GND
- net PVDD: no longer C1.1, C2.1
- net SH_A: now also C9.2, IC1.SH_A
- net VCC5V0: now also JP5.6
Other:
- moved on the sheet: C3, C4, TP1, TP2, TP3, TP4, U1, U4
Changed lines of the file:
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@@
 <?xml version="1.0" encoding="utf-8"?>
 <!DOCTYPE eagle SYSTEM "eagle.dtd">
-<eagle version="6.5.0">
+<eagle version="6.4">
 <drawing>
 <settings>
@@
 <part name="JP7" library="pavlo" deviceset="M03" device="-SCREW-5MM"/>
 <part name="SJ1" library="jumper" deviceset="SJ" device=""/>
-<part name="C1" library="ASL" deviceset="CAP" device="0805" value=".1 uF 100V"/>
-<part name="C2" library="ASL" deviceset="CAP" device="0805" value="2.2uF 100V"/>
 <part name="C3" library="ASL" deviceset="CAP" device="0805" value=".1 uF 100V"/>
 <part name="C4" library="ASL" deviceset="CAP" device="0805" value="2.2 uF"/>
@@
 </segment>
 </net>
-<net name="VCC5V" class="0">
+<net name="VCC5V0" class="0">
 <segment>
 <pinref part="JP5" gate="G$1" pin="6"/>
@@
 <instance part="C18" gate="G$1" x="162.06" y="122.12" rot="R180"/>
 <instance part="C19" gate="G$1" x="177.3" y="111.96" rot="R180"/>
-<instance part="C1" gate="G$1" x="355" y="203.8" smashed="yes">
-<attribute name="NAME" x="356.524" y="206.721" size="1.778" layer="95"/>
-<attribute name="VALUE" x="341.284" y="201.641" size="1.778" layer="96"/>
+<instance part="C3" gate="G$1" x="234.3" y="193.84" smashed="yes">
+<attribute name="NAME" x="235.824" y="196.761" size="1.778" layer="95"/>
+<attribute name="VALUE" x="220.584" y="191.681" size="1.778" layer="96"/>
 </instance>
-<instance part="C2" gate="G$1" x="364" y="204" smashed="yes">
-<attribute name="NAME" x="365.524" y="206.921" size="1.778" layer="95"/>
-<attribute name="VALUE" x="357.904" y="214.541" size="1.778" layer="96"/>
-</instance>
-<instance part="C3" gate="G$1" x="374" y="204" smashed="yes">
-<attribute name="NAME" x="375.524" y="206.921" size="1.778" layer="95"/>
-<attribute name="VALUE" x="370.444" y="194.221" size="1.778" layer="96"/>
-</instance>
-<instance part="C4" gate="G$1" x="381" y="204" smashed="yes">
-<attribute name="NAME" x="382.524" y="206.921" size="1.778" layer="95"/>
-<attribute name="VALUE" x="382.524" y="201.841" size="1.778" layer="96"/>
+<instance part="C4" gate="G$1" x="241.3" y="193.84" smashed="yes">
+<attribute name="NAME" x="242.824" y="196.761" size="1.778" layer="95"/>
+<attribute name="VALUE" x="242.824" y="191.681" size="1.778" layer="96"/>
 </instance>
 <instance part="FRAME2" gate="G$1" x="0" y="0"/>
 <instance part="FRAME2" gate="A" x="330" y="0"/>
-<instance part="TP1" gate="G$1" x="228.6" y="215.9"/>
-<instance part="TP2" gate="G$1" x="233.68" y="215.9"/>
-<instance part="TP3" gate="G$1" x="238.76" y="215.9"/>
-<instance part="TP4" gate="G$1" x="243.84" y="215.9"/>
+<instance part="TP1" gate="G$1" x="193.04" y="198.12"/>
+<instance part="TP2" gate="G$1" x="198.12" y="198.12"/>
+<instance part="TP3" gate="G$1" x="203.2" y="198.12"/>
+<instance part="TP4" gate="G$1" x="208.28" y="198.12"/>
 <instance part="TP6" gate="G$1" x="184.15" y="170.434" rot="R90"/>
 <instance part="TP7" gate="G$1" x="184.15" y="167.894" rot="R90"/>
@@
 </segment>
 <segment>
-<pinref part="C1" gate="G$1" pin="2"/>
-<wire x1="355" y1="201.26" x2="355" y2="201" width="0.1524" layer="91"/>
-<pinref part="C2" gate="G$1" pin="2"/>
-<wire x1="364" y1="201.46" x2="364" y2="201" width="0.1524" layer="91"/>
-<wire x1="355" y1="201" x2="364" y2="201" width="0.1524" layer="91"/>
-<wire x1="374" y1="201" x2="374" y2="201.46" width="0.1524" layer="91"/>
+<wire x1="234.3" y1="190.84" x2="234.3" y2="191.3" width="0.1524" layer="91"/>
 <pinref part="C3" gate="G$1" pin="2"/>
-<wire x1="364" y1="201" x2="374" y2="201" width="0.1524" layer="91"/>
-<wire x1="381" y1="201" x2="381" y2="201.46" width="0.1524" layer="91"/>
+<wire x1="241.3" y1="190.84" x2="241.3" y2="191.3" width="0.1524" layer="91"/>
 <pinref part="C4" gate="G$1" pin="2"/>
-<wire x1="374" y1="201" x2="381" y2="201" width="0.1524" layer="91"/>
-<label x="365" y="198" size="1.778" layer="95"/>
+<label x="231.904" y="187.84" size="1.778" layer="95"/>
+<wire x1="234.3" y1="190.84" x2="241.3" y2="190.84" width="0.1524" layer="91"/>
 </segment>
 <segment>
@@
 <net name="PVDD" class="3">
 <segment>
-<pinref part="C1" gate="G$1" pin="1"/>
-<wire x1="355" y1="208.88" x2="355" y2="210" width="0.1524" layer="91"/>
-<pinref part="C2" gate="G$1" pin="1"/>
-<wire x1="364" y1="209.08" x2="364" y2="210" width="0.1524" layer="91"/>
-<wire x1="355" y1="210" x2="364" y2="210" width="0.1524" layer="91"/>
 <pinref part="C3" gate="G$1" pin="1"/>
-<wire x1="374" y1="209.08" x2="374" y2="210" width="0.1524" layer="91"/>
-<wire x1="364" y1="210" x2="374" y2="210" width="0.1524" layer="91"/>
+<wire x1="234.3" y1="198.92" x2="234.3" y2="199.84" width="0.1524" layer="91"/>
 <pinref part="C4" gate="G$1" pin="1"/>
-<wire x1="381" y1="209.08" x2="381" y2="210" width="0.1524" layer="91"/>
-<wire x1="374" y1="210" x2="381" y2="210" width="0.1524" layer="91"/>
-<label x="365" y="211" size="1.778" layer="95"/>
+<wire x1="241.3" y1="198.92" x2="241.3" y2="199.84" width="0.1524" layer="91"/>
+<wire x1="234.3" y1="199.84" x2="241.3" y2="199.84" width="0.1524" layer="91"/>
+<label x="234.444" y="200.078" size="1.778" layer="95"/>
 </segment>
 <segment>
@@
 <segment>
 <pinref part="TP4" gate="G$1" pin="TP"/>
-<wire x1="243.84" y1="213.36" x2="243.84" y2="210.82" width="0.1524" layer="91"/>
-<label x="241.3" y="208.28" size="1.778" layer="95"/>
+<wire x1="208.28" y1="195.58" x2="208.28" y2="193.04" width="0.1524" layer="91"/>
+<label x="205.74" y="190.5" size="1.778" layer="95"/>
 </segment>
 </net>
@@
 <segment>
 <pinref part="TP1" gate="G$1" pin="TP"/>
-<wire x1="228.6" y1="213.36" x2="228.6" y2="210.82" width="0.1524" layer="91"/>
-<label x="226.06" y="205.74" size="1.778" layer="95"/>
+<wire x1="193.04" y1="195.58" x2="193.04" y2="193.04" width="0.1524" layer="91"/>
+<label x="190.5" y="187.96" size="1.778" layer="95"/>
 </segment>
 </net>
@@
 <segment>
 <pinref part="TP2" gate="G$1" pin="TP"/>
-<wire x1="233.68" y1="213.36" x2="233.68" y2="210.82" width="0.1524" layer="91"/>
-<label x="231.14" y="208.28" size="1.778" layer="95"/>
+<wire x1="198.12" y1="195.58" x2="198.12" y2="193.04" width="0.1524" layer="91"/>
+<label x="195.58" y="190.5" size="1.778" layer="95"/>
 </segment>
 </net>
@@
 <segment>
 <pinref part="TP3" gate="G$1" pin="TP"/>
-<wire x1="238.76" y1="213.36" x2="238.76" y2="210.82" width="0.1524" layer="91"/>
-<label x="236.22" y="205.74" size="1.778" layer="95"/>
+<wire x1="203.2" y1="195.58" x2="203.2" y2="193.04" width="0.1524" layer="91"/>
+<label x="200.66" y="187.96" size="1.778" layer="95"/>
 </segment>
 </net>
@@
 </segment>
 </net>
-<net name="N$11" class="0">
+<net name="SH_A" class="0">
 <segment>
 <pinref part="IC1" gate="G$1" pin="SH_A"/>
@@
 </segment>
 </net>
-<net name="GND" class="0">
+<net name="PGND" class="3">
 <segment>
 <pinref part="C5" gate="G$1" pin="2"/>

Commit message: More redesign work for v1.7
Parts:
- removed J2: (no value), ASL:M02PTH4
- removed JP1, JP2: (no value), ASL:M06SIP
- removed JP5: (no value), CMPE118lib:M06LOCK
- removed JP6: M03LOCK, ASL:M03LOCK
- removed JP7: M03-SCREW-5MM, pavlo:M03-SCREW-5MM
- removed JP8: (no value), ASL:M06SIP_LOCK
- added U$14, U$19: MICROCLASP3, OpenPMSM:MICROCLASP3
- added U$15: 3M10PIN2500, OpenPMSM:3M10PIN2500
- added U$16: MINIFITJR4PIN, OpenPMSM:MINIFITJR4PIN
- added U$17: MINIFITJR6PIN, OpenPMSM:MINIFITJR6PIN
- added U$18: MICROCLASP2, OpenPMSM:MICROCLASP2
- added U$20: MICROCLASP5, OpenPMSM:MICROCLASP5
Connections:
- net AN4: no longer JP5.4
- net AN5: no longer JP5.5
- net CAN_H: no longer JP6.2
- net CAN_L: no longer JP6.1
- net EN_A+: no longer JP8.2
- net EN_A-: no longer JP8.1
- net EN_B+: no longer JP8.3
- net EN_B-: no longer JP8.4
- net EN_C+: no longer JP8.6
- net EN_C-: no longer JP8.5
- net GND: no longer JP2.6, JP5.2, JP6.3
- net N$48: no longer JP1.6
- net N$49: no longer JP1.5
- net N$50: no longer JP1.4
- net N$51: no longer JP1.3
- net N$52: no longer JP1.2
- net N$53: no longer JP1.1
- net N$55: no longer JP2.2
- net N$56: no longer JP2.3
- net N$57: no longer JP2.4
- net N$58: no longer JP2.5
- net PGND: no longer J2.2
- net PVDD: no longer J2.1, JP2.1
- net RA11: no longer JP5.3
- net SH_A: no longer JP7.3
- net SH_B: no longer JP7.2
- net SH_C: no longer JP7.1
- net VCC3V3: no longer JP5.1
- net VCC5V0: no longer JP5.6

Commit message: Almost done with v1.7~
Parts:
- removed SJ4, SJ5, SJ6, SJ7: (no value), jumper:SJ
- removed U$1: DSPIC33EP128MC502-I/SS, pavlo:DSPIC33EP256MC50
- added U6: DSPIC33EP256MU80, OpenPMSM:DSPIC33EP256MU80
Connections:
- removed net AN4: U$1.PGEC1/AN4/C1IN1+/RPI34/RB2
- removed net AN5: U$1.PGED1/AN5/C1IN1-/RP35/RB3
- removed net EN_A: U$1.SDA1/RPI52/RC4, U3.ROUT1
- removed net EN_A+: U3.RIN1+
- removed net EN_A-: U3.RIN1
- removed net EN_B: U$1.SCK1/RPI51/RC3, U3.ROUT2
- removed net EN_B+: U3.RIN2+
- removed net EN_B-: U3.RIN2
- removed net EN_C: U$1.SDI1/RPI25/RA9, U3.ROUT3
- removed net EN_C+: U3.RIN3+
- removed net EN_C-: U3.RIN3
- removed net N$26: U$1.SCL1/RPI53/RC5
- removed net N$27: SJ4.2, U$1.RP118/RG6
- removed net N$28: SJ5.2, U$1.RPI119/RG7
- removed net N$29: SJ6.2, U$1.RP120/RG8
- removed net N$30: SJ7.2, U$1.RPI121/RG9
- removed net N$33: RN1.1, U$1.TCK/CVREF1O/ASCL1/RP40/T4CK/RB8
- removed net N$41: RN1.2, U$1.RC13
- removed net N$42: RN1.3, U$1.RP39/INT0/RB7
- removed net N$43: RN1.4, U$1.RPI58/RC10
- removed net N$48: U$1.FLT32/SCL2/RP36/RB4
- removed net N$49: U$1.SDA2/RPI24/RA8
- removed net N$50: U$1.AN15/RPI95/RE15
- removed net N$51: U$1.AN14/RPI94/RE14
- removed net N$52: U$1.AN13/C3IN2-/*U2CTS/RE13
- removed net N$53: U$1.AN12/C2IN2-/*U2RTS/BCLK2/RE12
- removed net N$55: U$1.PGEC3/VREF+/AN3/OA1OUT/RPI33/CTED1/RB1
- removed net N$56: U$1.AN6/OA3OUT/C4IN1+/OCFB/RC0
- removed net N$57: U$1.AN7/C3IN1-/C4IN1-/RC1
- removed net N$58: U$1.AN8/C3IN1+/*U1RTS/BCLK1/FLT3/RC2
- removed net RA11: U$1.AN9/RPI27/RA11
- removed net RA12: U$1.AN10/RPI28/RA12
- removed net RC9: U$1.RP57/RC9
- new net CH_A+: U$15.6, U3.RIN3+
- new net CH_A-: U$15.5, U3.RIN3
- new net CH_B+: U$15.4, U3.RIN2+
- new net CH_B-: U$15.3, U3.RIN2
- new net CH_I+: U$15.2, U3.RIN1+
- new net CH_I-: U$15.1, U3.RIN1
- new net HALL1: U$20.3, U6.ASCL1/PMCS2/RPI74/RD10
- new net HALL2: U$20.4, U6.ASDA1/DPLN/RPI73/RD9
- new net HALL3: U$20.5, U6.RTCC/DMLN/RPI72/RD8
- new net LED1: RN1.4, U6.AN8/PMA6/RPI40/RB8
- new net LED2: RN1.3, U6.AN9/PMA7//RPI41/RB9
- new net LED3: RN1.2, U6.TMS/AN10/CVREF/PMA13/RPI42/RB10
- new net LED4: RN1.1, U6.TDO/AN11/PMA12/RPI43/RB11
- new net QEI_A: U3.ROUT1, U6.C3IN1+/VCMPST3/RP71/RD7
- new net QEI_B: U3.ROUT2, U6.C3IN2-/RP70/RD6
- new net QEI_I: U3.ROUT3, U6.PMRD/RP69/RD5
- net *SCS: now also U6.C2IN1-/PMA2/RPI121/RG9; no longer U$1.RP56/RC8
- net CANRX: now also U6.SDA2/PMA9/RP100/RF4; no longer U$1.RPI96/RF0
- net CANTX: now also U6.SCL2/PMA8/RP101/RF5; no longer U$1.RP97/RF1
- net CRNT1: now also U6.TCK/AN12/PMA11/RPI44/RB12; no longer U$1.AN0/OA2OUT/RA0
- net CRNT2: now also U6.TDI/AN13/PMA10/RPI45/RB13; no longer U$1.AN1/C2IN1+/RA1
- net DC_CAL: now also U6.C2IN3-/SDO2/PMA3/RP120/RG8; no longer U$1.RD5
- net EN_GATE: now also U6.C1IN1-/SDI2/PMA4/RPI119/RG7; no longer U$1.RD6
- net GND: now also U$15.7, U$20.2, U6.AVSS, U6.VSS, U6.VSS_2, U6.VSS_3; no longer U$1.AVSS, U$1.VSS, U$1.VSS_2, U$1.VSS_3
- net MCLR: now also U6.*MCLR; no longer U$1.*MCLR
- net MISO: now also U6.AN31/PWM4H/PMD7/RP87/RE7; no longer U$1.RP54/RC6
- net MOSI: now also U6.C1IN3-/SCK2/PMA5/RP118/RG6; no longer U$1.RP55/RC7
- net N$25: now also U6.PGEC3/AN1/VREF-/RPI33/RB1; no longer U$1.PGED3/VREF-/AN2/C2IN1-/*SS1/RPI32/CTED2/RB0
- net N$31: now also U6.VCAP; no longer U$1.VCAP
- net N$5: now also U6.VDD_4; no longer SJ1.2, U$1.TDI/RA7
- net PGC: now also U6.PGED1/AN7/RCV/RPI39/RB7; no longer U$1.PGEC2/ASCL2/RP38/RB6
- net PGD: now also U6.PGEC1/AN6/RPI38/RB6; no longer U$1.PGED2/ASDA2/RP37/RB5
- net PWM1H: now also U6.AN29/PWM3H/PMD5/RP85/RE5; no longer U$1.RPI46/PWM1H/T3CK/RB14
- net PWM1L: now also U6.AN28/PWM3L/PMD4/RP84/RE4; no longer U$1.RPI47/PWM1L/T5CK/RB15
- net PWM2H: now also U6.AN27/PWM2H/PMD3/RPI83/RE3; no longer U$1.RPI44/PWM2H/RB12
- net PWM2L: now also U6.AN26/PWM2L/PMD2/RP82/RE2; no longer U$1.RPI45/PWM2L/CTPLS/RB13
- net PWM3H: now also U6.AN25/PWM1H/PMD1/RPI81/RE1; no longer U$1.RP42/PWM3H/RB10
- net PWM3L: now also U6.AN24/PWM1L/PMD0/RP80/RE0; no longer U$1.RB43/PWM3L/RB11
- net SCLK: now also U6.AN30/PWM4L/PMD6/RPI86/RE6; no longer U$1.TMS/ASDA1/RP41/RB9
- net VCC3V3: now also U$20.1, U6.AVDD, U6.VDD, U6.VDD_2, U6.VDD_3; no longer SJ1.1, SJ4.1, SJ5.1, SJ6.1, SJ7.1, U$1.AVDD, U$1.VDD, U$1.VDD_2, U$1.VDD_3, U$1.VDD_4
- net VCC5V0: now also U$15.10
Other:
- moved on the sheet: C20, RN1, SJ1
