File: PMSM Board v1.7/Eagle Files/CANTensegrityBoard.brd (EAGLE design)
At the start: 100.5 x 48 mm, 98 parts, among them IC1 DRV8303, U1 TPS73733-Q1_DRB_8, U10 H1206T500R-10, U2 SN65HVD232_D_8, U3 SN65LVDT348_PW_1, U4 TPS54240_DRC_10, U5 LP38692_NGG_6, U6 DSPIC33EP256MU80, U9 H1206T500R-10

Commit message: Choring up code for v1.7.
Connections:
- removed net N$5: U6.38
- net PGC: now also U6.17; no longer U6.18
- net PGD: now also U6.18; no longer U6.17
- net VCC3V3: now also U6.38
Routing:
- net VCC3V3: track 98.5 -> 102.7 mm, vias 12 -> 13
- net PGC: track 25.4 -> 23.4 mm
Changed lines of the file:
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@@
 <?xml version="1.0" encoding="utf-8"?>
 <!DOCTYPE eagle SYSTEM "eagle.dtd">
-<eagle version="6.4">
+<eagle version="6.5.0">
 <drawing>
 <settings>
@@
 <signal name="PGD" class="2">
 <contactref element="JP3" pad="4"/>
-<contactref element="U6" pad="17"/>
-<wire x1="28.2592" y1="29.5134" x2="28.26" y2="29.5126" width="0.2032" layer="1"/>
 <wire x1="28.26" y1="29.5126" x2="28.26" y2="27.16" width="0.2032" layer="1"/>
 <wire x1="28.26" y1="27.16" x2="27.9" y2="26.8" width="0.2032" layer="1"/>
@@
 <wire x1="27.5" y1="25.8" x2="27.9" y2="26.2" width="0.2032" layer="1"/>
 <wire x1="27.1" y1="25.8" x2="26.7" y2="25.8" width="0.2032" layer="15"/>
+<contactref element="U6" pad="18"/>
+<wire x1="28.26" y1="29.5126" x2="27.7512" y2="29.5134" width="0" layer="19" extent="1-1"/>
 </signal>
 <signal name="PGC">
 <contactref element="JP3" pad="5"/>
-<contactref element="U6" pad="18"/>
-<wire x1="27.7512" y1="29.5134" x2="27.7512" y2="27.5512" width="0.2032" layer="1"/>
 <wire x1="27.7512" y1="27.5512" x2="27.1" y2="26.9" width="0.2032" layer="1"/>
 <via x="27.1" y="26.9" extent="1-16" drill="0.4" shape="square"/>
@@
 <wire x1="19.4" y1="46.057" x2="19.47" y2="46.127" width="0.254" layer="15"/>
 <wire x1="19.47" y1="44.03" x2="19.47" y2="46.127" width="0.2032" layer="15"/>
+<contactref element="U6" pad="17"/>
+<wire x1="27.7512" y1="27.5512" x2="28.2592" y2="29.5134" width="0" layer="19" extent="1-1"/>
 </signal>
 <signal name="VCC3V3" class="3">
@@
 <wire x1="16.0198" y1="17.4198" x2="15.8" y2="17.6" width="0.3048" layer="1"/>
 <contactref element="JP1" pad="6"/>
+<contactref element="U6" pad="38"/>
+<wire x1="18.8866" y1="25.1446" x2="17.8554" y2="25.1446" width="0.2032" layer="1"/>
+<via x="16" y="27.5" extent="1-16" drill="0.4" shape="square"/>
+<wire x1="16" y1="27.5" x2="16" y2="27" width="0.2032" layer="1"/>
+<wire x1="16" y1="27" x2="17.8554" y2="25.1446" width="0.2032" layer="1"/>
 </signal>
 <signal name="N$31">
@@
 <wire x1="26.6" y1="34.9" x2="26.6" y2="36.05" width="0.254" layer="1"/>
 </signal>
-<signal name="N$5">
-<contactref element="U6" pad="38"/>
-</signal>
 <signal name="QEI_A">

Commit message: Started board version 1.8
Parts:
- removed C14: 5600pF, SwitcherPowerStage:0805
- removed C15: 270pF, SwitcherPowerStage:0805
- removed C29: 47uF\, SwitcherPowerStage:C2220K
- removed C30, C31, C32: 1uF, SwitcherPowerStage:0805
- removed C8: .1uF, SwitcherPowerStage:0805
- removed D1: DIODE-SCHOTTKY240A, SwitcherPowerStage:SMA-DIODE-B240A
- removed R10: 59k, SwitcherPowerStage:0805
- removed R11: 10k, SwitcherPowerStage:0805
- removed R2: 348k, SwitcherPowerStage:0805
- removed R3: 88.7k, SwitcherPowerStage:0805
- removed R8: 237k, SwitcherPowerStage:0805
- removed R9: 7.68k, SwitcherPowerStage:0805
- removed U$13: SLF12555T, SwitcherPowerStage:SLF12555
- removed U1: TPS73733-Q1_DRB_8, SwitcherPowerStage:DRB8_1P75X1P5
- removed U4: TPS54240_DRC_10, SwitcherPowerStage:DRC10_2P4X1P65
- removed U5: LP38692_NGG_6, SwitcherPowerStage:SDE06A
- added C1, C38: 1uF, SensorCape:0805
- added C2, C33, C34, C35, C36, C37, C39, C50, C51, C52, C53, C54: 10uF, SensorCape:0805
- added C40, C45: 22uF, SensorCape:1210
- added C41, C43: 2.2uF 100V, SensorCape:1210
- added C42: 27uF 100V, SensorCape:CPOL-RADIAL-100UF-25V
- added C47: 10nF, SensorCape:0805
- added R24: 48.7, ASL:0805
- added R25: 1100k, ASL:0805
- added R26: 174k, ASL:0805
- added R27: 40.2k, ASL:0805
- added U$1, U$22: TPS7A4700_RGW_20, SensorCape:RGW20_3P15X3P15
- added U7: TPS84250_RKG_41, SensorCape:RKG41
- C5: value 4.7uF -> 2.2uF 100V; device SwitcherPowerStage:1210 -> SensorCape:1210
- C6: value .01uF -> 22uF; device SwitcherPowerStage:0805 -> SensorCape:1210
- moved C5 20.6 mm to (62.0, 29.5), turned to 0 degrees
- moved C6 15.8 mm to (48.5, 45.0), turned to 90 degrees
Connections:
- removed net N$10: C8.1, U4.1
- removed net N$13: C8.2, D1.C, U$13.P$1, U4.10
- removed net N$14: C15.1, R9.2, U4.8
- removed net N$15: C14.1, R9.1
- removed net N$16: R10.1, R11.2, U4.7
- removed net N$7: R2.1, R3.2, U4.3
- removed net N$8: C6.1, U4.4
- removed net N$9: R8.2, U4.5
- new net N$23: C38.1, U$22.14
- new net N$37: R24.1, U7.36
- new net N$38: R25.2, U7.31
- new net N$41: R26.1, R27.2, U7.27
- new net N$43: C47.1, U7.28
- new net N$5: C1.1, U$1.14
- net PGND: now also C1.2, C2.2, C33.2, C34.2, C35.2, C36.2, C37.2, C38.2, C39.2, C40.1, C41.2, C42.2, C43.2, C45.1, C47.2, C50.2, C51.2, C52.2, C53.2, C54.2, C6.1, R25.1, R27.1, U$1.10, U$1.21, U$1.6, U$1.7, U$22.11, U$22.12, U$22.21, U$22.7, U$22.8, U7.1, U7.16, U7.17, U7.18, U7.19, U7.20, U7.29, U7.30, U7.32, U7.33, U7.34, U7.37, U7.4, U7.40, U7.5, U7.8, U7.9; no longer C14.2, C15.2, C29.2, C30.2, C31.2, C32.2, C6.2, D1.A, R11.1, R3.1, R8.1, U1.4, U1.9, U1.P$1, U1.P$2, U1.P$3, U1.P$4, U4.9, U5.2, U5.7
- net PVDD: now also C41.1, C42.1, C43.1, R26.2, U7.26; no longer R2.2, U4.2
- net VCC3V3: now also C39.1, C50.1, C51.1, C52.1, C53.1, U$22.1, U$22.20, U$22.3; no longer C32.1, U1.1
- net VCC5V0: now also C2.1, C33.1, C34.1, C35.1, C36.1, C54.1, U$1.1, U$1.20, U$1.3, U$22.13, U$22.15, U$22.16; no longer C31.1, U1.5, U1.8, U5.4, U5.5
- net VCC5V5: now also C37.1, C40.2, C45.2, C6.2, R24.2, U$1.13, U$1.15, U$1.16, U7.10, U7.11, U7.12, U7.13, U7.14, U7.15, U7.39; no longer C29.1, C30.1, R10.2, U$13.P$2, U5.1, U5.3, U5.6
Routing:
- net VCC5V5: track 50.4 -> 7.25 mm, vias 2 -> 6
- net N$13: track 25.4 -> 0.00 mm, vias 2 -> 0
- net N$16: track 16.0 -> 0.00 mm
- net VCC5V0: track 9.62 -> 0.00 mm, vias 2 -> 0
- net PGND: track 13.7 -> 5.08 mm, vias 33 -> 24
- net N$7: track 7.79 -> 0.00 mm
- net PVDD: track 50.0 -> 42.3 mm, vias 6 -> 2
- net N$14: track 4.74 -> 0.00 mm
- net VCC3V3: track 102.7 -> 97.9 mm, vias 13 -> 11
- net N$10: track 4.63 -> 0.00 mm
- net N$8: track 3.60 -> 0.00 mm
- net N$15: track 2.11 -> 0.00 mm
- net N$9: track 1.54 -> 0.00 mm
