File: PMSM Board v1.7/Eagle Files/CANTensegrityBoard.sch (EAGLE design)
At the start: 94 parts, among them IC1 DRV8303, U1 TPS73733-Q1_DRB_8, U10 H1206T500R-10, U2 SN65HVD232_D_8, U3 SN65LVDT348_PW_1, U4 TPS54240_DRC_10, U5 LP38692_NGG_6, U6 DSPIC33EP256MU80, U9 H1206T500R-10

Commit message: Started board version 1.8
Parts:
- removed C14: 5600pF, SwitcherPowerStage:CAP0805
- removed C15: 270pF, SwitcherPowerStage:CAP0805
- removed C29: 47uF\, SwitcherPowerStage:CAP
- removed C30, C31, C32: 1uF, SwitcherPowerStage:CAP0805
- removed C8: .1uF, SwitcherPowerStage:CAP0805
- removed D1: DIODE-SCHOTTKY240A, SwitcherPowerStage:DIODE-SCHOTTKY240A
- removed R10: 59k, SwitcherPowerStage:RESISTOR0805-RES
- removed R11: 10k, SwitcherPowerStage:RESISTOR0805-RES
- removed R2: 348k, SwitcherPowerStage:RESISTOR0805-RES
- removed R3: 88.7k, SwitcherPowerStage:RESISTOR0805-RES
- removed R8: 237k, SwitcherPowerStage:RESISTOR0805-RES
- removed R9: 7.68k, SwitcherPowerStage:RESISTOR0805-RES
- removed U$13: SLF12555T, SwitcherPowerStage:SLF12555T
- removed U1: TPS73733-Q1_DRB_8, SwitcherPowerStage:TPS73733-Q1_DRB_8
- removed U4: TPS54240_DRC_10, SwitcherPowerStage:TPS54240_DRC_10
- removed U5: LP38692_NGG_6, SwitcherPowerStage:LP38692_NGG_6
- added C1, C38: 1uF, SensorCape:CAP0805
- added C2, C33, C34, C35, C36, C37, C39, C50, C51, C52, C53, C54: 10uF, SensorCape:CAP0805
- added C40, C45: 22uF, SensorCape:CAP1210
- added C41, C43: 2.2uF 100V, SensorCape:CAP1210
- added C42: 27uF 100V, SensorCape:CAP_POLPTH1
- added C47: 10nF, SensorCape:CAP0805
- added R24: 48.7, ASL:RESISTOR0805-RES
- added R25: 1100k, ASL:RESISTOR0805-RES
- added R26: 174k, ASL:RESISTOR0805-RES
- added R27: 40.2k, ASL:RESISTOR0805-RES
- added U$1, U$22: TPS7A4700_RGW_20, SensorCape:TPS7A4700_RGW_20
- added U7: TPS84250_RKG_41, SensorCape:TPS84250_RKG_41
- C5: value 4.7uF -> 2.2uF 100V; device SwitcherPowerStage:CAP1210 -> SensorCape:CAP1210
- C6: value .01uF -> 22uF; device SwitcherPowerStage:CAP0805 -> SensorCape:CAP1210
Connections:
- removed net N$10: C8.1, U4.BOOT
- removed net N$13: C8.2, D1.C, U$13.1, U4.PH
- removed net N$14: C15.1, R9.2, U4.COMP
- removed net N$15: C14.1, R9.1
- removed net N$16: R10.1, R11.2, U4.VSENSE
- removed net N$7: R2.1, R3.2, U4.EN
- removed net N$8: C6.1, U4.SS/TR
- removed net N$9: R8.2, U4.RT/CLK
- new net N$23: C38.1, U$22.NR
- new net N$37: R24.1, U7.VADJ
- new net N$38: R25.2, U7.RT/CLK
- new net N$41: R26.1, R27.2, U7.INH/UVLO
- new net N$43: C47.1, U7.SS/TR
- new net N$5: C1.1, U$1.NR
- net PGND: now also C1.2, C2.2, C33.2, C34.2, C35.2, C36.2, C37.2, C38.2, C39.2, C40.1, C41.2, C42.-, C43.2, C45.1, C47.2, C50.2, C51.2, C52.2, C53.2, C54.2, C6.1, R25.1, R27.1, U$1.0P4V, U$1.3P2V, U$1.EPAD, U$1.GND, U$22.0P1V, U$22.0P2V, U$22.1P6V, U$22.EPAD, U$22.GND, U7.AGND, U7.GND_PT, U7.PGND, U7.STSEL; no longer C14.2, C15.2, C29.2, C30.2, C31.2, C32.2, C6.2, D1.A, R11.1, R3.1, R8.1, U1.EPAD, U1.GND, U4.GND, U5.7, U5.GND
- net PVDD: now also C41.1, C42.+, C43.1, R26.2, U7.VIN; no longer R2.2, U4.VIN
- net VCC3V3: now also C39.1, C50.1, C51.1, C52.1, C53.1, U$22.OUT, U$22.OUT_1, U$22.SENSE/FB; no longer C32.1, U1.OUT
- net VCC5V0: now also C2.1, C33.1, C34.1, C35.1, C36.1, C54.1, U$1.OUT, U$1.OUT_1, U$1.SENSE/FB, U$22.EN, U$22.IN, U$22.IN_2; no longer C31.1, U1.EN, U1.IN, U5.SNS, U5.VOUT
- net VCC5V5: now also C37.1, C40.2, C45.2, C6.2, R24.2, U$1.EN, U$1.IN, U$1.IN_2, U7.VOUT; no longer C29.1, C30.1, R10.2, U$13.2, U5.VEN, U5.VIN, U5.VIN_2
