File: PMSM Board v1.9b/Eagle Files/CANTensegrityBoard.sch (EAGLE design)
At the start: 115 parts, among them IC1 DRV8303, U2 SN65HVD232_D_8, U3 SN65LVDT348_PW_1, U6 DSPIC33EP256MU80, U7 TPS84250_RKG_41

Commit message: Lots of FOC work.
Parts:
- R14, R15: value (none) -> 1k
Changed lines of the file:
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@@
 <part name="U6" library="OpenPMSM" deviceset="DSPIC33EP256MU80" device=""/>
 <part name="R12" library="ASL" deviceset="RESISTOR" device="0805-RES" value="10k"/>
-<part name="R14" library="ASL" deviceset="RESISTOR" device="0805-RES"/>
-<part name="R15" library="ASL" deviceset="RESISTOR" device="0805-RES"/>
+<part name="R14" library="ASL" deviceset="RESISTOR" device="0805-RES" value="1k"/>
+<part name="R15" library="ASL" deviceset="RESISTOR" device="0805-RES" value="1k"/>
 <part name="LED5" library="ASL" deviceset="LED" device="0805"/>
 <part name="LED6" library="ASL" deviceset="LED" device="0805"/>
